File: Hackpad.kicad_pcb (KiCad board)
At the start: 2 copper layers, 99 x 70 mm, 14 parts, among them SW1 SW_Push, SW2 SW_Push, SW3 SW_Push, SW4 SW_Push, SW5 SW_Push, SW6 RotaryEncoder_Switch_MP, U1 XIAO-RP2040-DIP

Commit message: Add text
Other:
- board text added: "5V"
- board text added: "Click click"
- board text added: "FISH"
- board text added: "Fleny's hackpad Media"
- board text added: "Furries :3"
- board text added: "GND"
- board text added: "Ninja Tuna"
- board text added: "Oh Look Endless Doom"
- board text added: "SCL"
- board text added: "SDA"
- board text added: "Spinny spinny"
- board text added: "Swatch"
- board text added: "Swetch"
- board text added: "Switch"
- board text added: "Swotch"
- board text added: "Swuch"
- board text added: "USB C over here"
- board text added: "XIAO HERE"
- board text removed: "Fleny's pad"
- board text removed: "XIAO HERE!"
Changed lines of the file:
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@@
 		(tags "rotary encoder")
 		(property "Reference" "SW6"
-			(at 2.8 -4.7 0)
+			(at -2 7.5 0)
 			(layer "F.SilkS")
 			(effects
@@
 		(tags "CONN DEV")
 		(property "Reference" "OL1"
-			(at 0 2.25 90)
+			(at -6.75 -2.75 180)
 			(layer "F.Fab")
 			(effects
@@
 		(at 114.84 78.5)
 		(property "Reference" "U1"
-			(at -10.995 -6.2125 0)
+			(at 10.16 -9.5 0)
 			(unlocked yes)
 			(layer "F.SilkS")
-			(hide yes)
 			(effects
 				(font
@@
 		(layer "Edge.Cuts")
 	)
-	(gr_text "XIAO HERE!"
-		(at 110.49 84 0)
+	(gr_text "Swuch\n"
+		(at 141 131 0)
+		(layer "F.SilkS")
+		(effects
+			(font
+				(size 1 1)
+				(thickness 0.1)
+			)
+			(justify left bottom)
+		)
+	)
+	(gr_text "Spinny spinny"
+		(at 151 111 0)
 		(layer "F.SilkS")
 		(effects
@@
 		)
 	)
-	(gr_text "Fleny's pad"
-		(at 144 80.3 0)
+	(gr_text "5V"
+		(at 94 105.5 90)
+		(layer "F.SilkS")
+		(effects
+			(font
+				(size 1 1)
+				(thickness 0.2)
+				(bold yes)
+			)
+			(justify left bottom)
+		)
+	)
+	(gr_text "Click click"
+		(at 103.75 132.75 0)
+		(layer "F.SilkS")
+		(effects
+			(font
+				(size 1 1)
+				(thickness 0.1)
+			)
+			(justify left bottom)
+		)
+	)
+	(gr_text "GND"
+		(at 94 109.25 90)
+		(layer "F.SilkS")
+		(effects
+			(font
+				(size 1 1)
+				(thickness 0.2)
+				(bold yes)
+			)
+			(justify left bottom)
+		)
+	)
+	(gr_text "XIAO HERE"
+		(at 108 86 0)
+		(layer "F.SilkS")
+		(effects
+			(font
+				(size 1.7 1.7)
+				(thickness 0.4)
+				(bold yes)
+			)
+			(justify left bottom)
+		)
+	)
+	(gr_text "SDA"
+		(at 94 100 90)
+		(layer "F.SilkS")
+		(effects
+			(font
+				(size 1 1)
+				(thickness 0.2)
+				(bold yes)
+			)
+			(justify left bottom)
+		)
+	)
+	(gr_text "SCL"
+		(at 94 103.25 90)
+		(layer "F.SilkS")
+		(effects
+			(font
+				(size 1 1)
+				(thickness 0.2)
+				(bold yes)
+			)
+			(justify left bottom)
+		)
+	)
+	(gr_text "USB C over here"
+		(at 109 69.864001 0)
+		(layer "F.SilkS")
+		(effects
+			(font
+				(size 1 1)
+				(thickness 0.2)
+				(bold yes)
+			)
+			(justify left bottom)
+		)
+	)
+	(gr_text "Swatch"
+		(at 121 131 0)
+		(layer "F.SilkS")
+		(effects
+			(font
+				(size 1 1)
+				(thickness 0.1)
+			)
+			(justify left bottom)
+		)
+	)
+	(gr_text "Furries :3"
+		(at 93 114 0)
+		(layer "F.SilkS")
+		(effects
+			(font
+				(size 1.5 1.5)
+				(thickness 0.3)
+				(bold yes)
+			)
+			(justify left bottom)
+		)
+	)
+	(gr_text "Fleny's hackpad\nMedia\n"
+		(at 143 83 0)
+		(layer "F.SilkS")
+		(effects
+			(font
+				(size 1 1)
+				(thickness 0.2)
+				(bold yes)
+			)
+			(justify left bottom)
+		)
+	)
+	(gr_text "Oh\nLook\n\nEndless\nDoom"
+		(at 101.5 107.75 0)
 		(layer "F.SilkS")
 		(effects
@@
 			)
 			(justify left bottom)
+		)
+	)
+	(gr_text "5V"
+		(at 133 71 0)
+		(layer "F.SilkS")
+		(effects
+			(font
+				(size 1 1)
+				(thickness 0.2)
+				(bold yes)
+			)
+			(justify left bottom)
+		)
+	)
+	(gr_text "Swetch"
+		(at 77 107 0)
+		(layer "F.SilkS")
+		(effects
+			(font
+				(size 1 1)
+				(thickness 0.1)
+			)
+			(justify left bottom)
+		)
+	)
+	(gr_text "FISH"
+		(at 114 94 0)
+		(layer "F.SilkS")
+		(effects
+			(font
+				(size 0.8 0.8)
+				(thickness 0.1)
+			)
+			(justify left bottom)
+		)
+	)
+	(gr_text "Switch"
+		(at 83 131 0)
+		(layer "F.SilkS")
+		(effects
+			(font
+				(size 1 1)
+				(thickness 0.125)
+			)
+			(justify left bottom)
+		)
+	)
+	(gr_text "GND"
+		(at 131 74 0)
+		(layer "F.SilkS")
+		(effects
+			(font
+				(size 1 1)
+				(thickness 0.2)
+				(bold yes)
+			)
+			(justify left bottom)
+		)
+	)
+	(gr_text "Swotch"
+		(at 102 131 0)
+		(layer "F.SilkS")
+		(effects
+			(font
+				(size 1 1)
+				(thickness 0.1)
+			)
+			(justify left bottom)
+		)
+	)
+	(gr_text "Ninja Tuna"
+		(at 106 93 0)
+		(layer "F.SilkS")
+		(effects
+			(font
+				(size 2 2)
+				(thickness 0.25)
+			)
+			(justify left bottom)
